Commit message: 데탑 로컬 작업 스냅샷 — 원격 동기화 전 보존
base_map_h*.sdf, documents/, start_goal_markers.py 등 데탑에서만 있던 것과
display.rviz / navigation.launch.py / ekf.yaml 수정분을 기록으로 남긴다.
메시(STL)는 실제 파일로 들어간다 (.gitattributes 가 없어 LFS 필터 미적용).

File: src/drobot_description/urdf/drobot.urdf.xacro (robot description, xacro)
@@ -64,5 +64,5 @@
   </link>
   <joint name="lidar_joint" type="fixed">
-    <origin xyz="0.010101 -0.027788 0.30154" rpy="3.1416 0 3.1416"/>
+    <origin xyz="0.010101 -0.027788 0.30154" rpy="0 0 0"/>
     <parent link="base_link"/>
     <child link="lidar"/>

File: src/drobot_description/urdf/gazebo.xacro (robot description, xacro)
@@ -112,5 +112,5 @@
         <range>
           <min>0.5</min>
-          <max>12.0</max>
+          <max>20.0</max>
           <resolution>0.01</resolution>
         </range>

Commit message: description: 센서 프레임명을 인터페이스 규약에 맞춤 (lidar→base_scan, camera→camera_link)

File: src/drobot_description/urdf/drobot.urdf.xacro (robot description, xacro)
@@ -46,5 +46,5 @@
   </link>
   <!-- ==================== LIDAR ==================== -->
-  <link name="lidar">
+  <link name="base_scan">
     <inertial>
       <origin xyz="-0.0215847721606996 0.00397566854868606 -0.00218033584701988" rpy="0 0 0"/>
@@ -66,8 +66,8 @@
     <origin xyz="0.010101 -0.027788 0.30154" rpy="0 0 0"/>
     <parent link="base_link"/>
-    <child link="lidar"/>
+    <child link="base_scan"/>
   </joint>
   <!-- ==================== CAMERA ==================== -->
-  <link name="camera">
+  <link name="camera_link">
     <inertial>
       <origin xyz="-0.0215847721606996 0.00397566854868603 -0.00218033584701988" rpy="3.1416 0 3.1416"/>
@@ -89,5 +89,5 @@
     <origin xyz="0.010101 -0.027788 0.36" rpy="0 0 0"/>
     <parent link="base_link"/>
-    <child link="camera"/>
+    <child link="camera_link"/>
   </joint>
   <!-- ==================== IMU (virtual, no mesh) ==================== -->

File: src/drobot_description/urdf/drobot_primitives.urdf.xacro (robot description, xacro)
@@ -57,5 +57,5 @@
   </link>
   <!-- ==================== LIDAR ==================== -->
-  <link name="lidar">
+  <link name="base_scan">
     <inertial>
       <origin xyz="-0.0215847721606996 0.00397566854868606 -0.00218033584701988" rpy="0 0 0"/>
@@ -77,8 +77,8 @@
     <origin xyz="0.010101 -0.027788 0.30154" rpy="3.1416 0 3.1416"/>
     <parent link="base_link"/>
-    <child link="lidar"/>
+    <child link="base_scan"/>
   </joint>
   <!-- ==================== CAMERA ==================== -->
-  <link name="camera">
+  <link name="camera_link">
     <inertial>
       <origin xyz="-0.0215847721606996 0.00397566854868603 -0.00218033584701988" rpy="3.1416 0 3.1416"/>
@@ -100,5 +100,5 @@
     <origin xyz="0.010101 -0.027788 0.36" rpy="0 0 0"/>
     <parent link="base_link"/>
-    <child link="camera"/>
+    <child link="camera_link"/>
   </joint>
   <!-- ==================== IMU (virtual, no mesh) ==================== -->

File: src/drobot_description/urdf/gazebo.xacro (robot description, xacro)
@@ -94,8 +94,8 @@
   </gazebo>
   <!-- ========== 2D LIDAR ========== -->
-  <gazebo reference="lidar">
+  <gazebo reference="base_scan">
     <sensor name="lidar" type="gpu_lidar">
       <topic>/scan</topic>
-      <gz_frame_id>lidar</gz_frame_id>
+      <gz_frame_id>base_scan</gz_frame_id>
       <update_rate>10</update_rate>
       <always_on>true</always_on>
@@ -140,6 +140,6 @@
   </gazebo>
   <!-- ========== CAMERA ========== -->
-  <gazebo reference="camera">
-    <sensor name="camera" type="rgbd"> <gz_frame_id>camera</gz_frame_id>
+  <gazebo reference="camera_link">
+    <sensor name="camera" type="rgbd"> <gz_frame_id>camera_link</gz_frame_id>
       <update_rate>15</update_rate>
       <always_on>true</always_on>

Commit message: 데탑 로컬 작업 스냅샷 — 통합 전 보존 (B 트랙 테스트 포함)

File: src/drobot_description/urdf/drobot.urdf.xacro (robot description, xacro)
@@ -64,5 +64,5 @@
   </link>
   <joint name="lidar_joint" type="fixed">
-    <origin xyz="0.010101 -0.027788 0.30154" rpy="0 0 0"/>
+    <origin xyz="0.010101 -0.027788 0.30154" rpy="3.1416 0 3.1416"/>
     <parent link="base_link"/>
     <child link="lidar"/>

File: src/drobot_description/urdf/gazebo.xacro (robot description, xacro)
@@ -112,5 +112,5 @@
         <range>
           <min>0.5</min>
-          <max>20.0</max>
+          <max>12.0</max>
           <resolution>0.01</resolution>
         </range>

Commit message: A 트랙: 카메라 광학 프레임 추가 — 포인트클라우드 좌표가 통째로 어긋나 있었다
증상 (실측, /clock 퍼블리셔 1개·시간 역행 0 인 깨끗한 실행)
  elevation_layer 가 본 높이, x=2.12 선상
        실제            레이어
    y=1.95~4.05  0.00 m 빈 바닥   0.25 m  (전 구간 균일)
    y=4.20~6.00  0.50 m 장애물    미관측
  빈 바닥을 0.25 m 로 보고 진짜 장애물은 전혀 못 봤다.
  0.25 m 는 base_link 의 지면 높이다 (라이다 센서 원점 z=0.55,
  lidar_joint z=0.30154 -> base_link = 0.248). 지형이 아니라 로봇 자신이다.

원인
  Gazebo 의 rgbd 센서는 포인트클라우드를 광학 좌표계(x 우·y 하·z 전방)로
  낸다. 그런데 gz_frame_id 가 camera_link 였다 — ROS 본체 좌표계
  (x 전방·y 좌·z 상, REP-103). 축이 두 번 90도 어긋나 모든 점이 엉뚱한
  자리와 높이로 들어갔다. URDF 에 광학 프레임 자체가 없었다.

조치
  camera_link_optical 링크와 고정 조인트 추가 (rpy -pi/2 0 -pi/2),
  gz_frame_id 를 그쪽으로. drobot.urdf.xacro 와 primitives 양쪽.

왜 중요한가
  elevation_layer 가 유일하게 장애물을 볼 수 있는 센서가 깊이 카메라다.
  2D 라이다는 base_link+0.30154 = 지면 0.55 m 라 0.5 m 장애물 위로 지나간다
  (통제 맵 h0.05·h0.3·h0.5 세 개가 라이다에 원리적으로 안 보인다).
  카메라가 틀려 있으면 그 세 맵에서 지형 인지가 통째로 없는 셈이다.

File: src/drobot_description/urdf/drobot.urdf.xacro (robot description, xacro)
@@ -91,4 +91,20 @@
     <child link="camera_link"/>
   </joint>
+  <!-- 카메라 광학 프레임 (REP-103 / REP-145)
+       Gazebo 의 rgbd 센서는 포인트클라우드를 광학 좌표계로 낸다:
+           x 오른쪽 · y 아래 · z 전방
+       반면 camera_link 는 ROS 본체 좌표계다:
+           x 전방 · y 왼쪽 · z 위
+       둘을 같은 프레임으로 선언하면 축이 두 번 90도 어긋나, 바닥 점이
+       로봇 자신의 높이로 찍히고 장애물은 엉뚱한 자리에 쌓인다.
+       실제로 elevation_layer 가 빈 바닥 전 구간을 0.25 m(= base_link 높이)로
+       보고 0.5 m 장애물은 전혀 못 봤다. 2026-10-02 확인.
+       gazebo.xacro 의 gz_frame_id 가 이 프레임을 가리킨다. -->
+  <link name="camera_link_optical"/>
+  <joint name="camera_optical_joint" type="fixed">
+    <origin xyz="0 0 0" rpy="-1.5707963267948966 0 -1.5707963267948966"/>
+    <parent link="camera_link"/>
+    <child link="camera_link_optical"/>
+  </joint>
   <!-- ==================== IMU (virtual, no mesh) ==================== -->
   <link name="imu_link">

File: src/drobot_description/urdf/drobot_primitives.urdf.xacro (robot description, xacro)
@@ -114,4 +114,20 @@
     <child link="camera_link"/>
   </joint>
+  <!-- 카메라 광학 프레임 (REP-103 / REP-145)
+       Gazebo 의 rgbd 센서는 포인트클라우드를 광학 좌표계로 낸다:
+           x 오른쪽 · y 아래 · z 전방
+       반면 camera_link 는 ROS 본체 좌표계다:
+           x 전방 · y 왼쪽 · z 위
+       둘을 같은 프레임으로 선언하면 축이 두 번 90도 어긋나, 바닥 점이
+       로봇 자신의 높이로 찍히고 장애물은 엉뚱한 자리에 쌓인다.
+       실제로 elevation_layer 가 빈 바닥 전 구간을 0.25 m(= base_link 높이)로
+       보고 0.5 m 장애물은 전혀 못 봤다. 2026-10-02 확인.
+       gazebo.xacro 의 gz_frame_id 가 이 프레임을 가리킨다. -->
+  <link name="camera_link_optical"/>
+  <joint name="camera_optical_joint" type="fixed">
+    <origin xyz="0 0 0" rpy="-1.5707963267948966 0 -1.5707963267948966"/>
+    <parent link="camera_link"/>
+    <child link="camera_link_optical"/>
+  </joint>
   <!-- ==================== IMU (virtual, no mesh) ==================== -->
   <link name="imu_link">

File: src/drobot_description/urdf/gazebo.xacro (robot description, xacro)
@@ -141,5 +141,5 @@
   <!-- ========== CAMERA ========== -->
   <gazebo reference="camera_link">
-    <sensor name="camera" type="rgbd"> <gz_frame_id>camera_link</gz_frame_id>
+    <sensor name="camera" type="rgbd"> <gz_frame_id>camera_link_optical</gz_frame_id>
       <update_rate>15</update_rate>
       <always_on>true</always_on>

Commit message: URDF: base_footprint 높이 0.25 -> 0 — 빈 바닥이 0.25m 로 보이던 원인
메시 모델은 base_link 원점이 이미 바닥 높이다 (바퀴 접지점 base_link 기준 -0.002/+0.005).
0.25 오프셋 때문에 Gazebo 에서 base_footprint 가 땅 밑 -0.25m 에 놓였고
(gz model z = -0.2518 실측), EKF two_d_mode 가 이를 z=0 으로 고정해
TF 를 거친 센서 점이 전부 0.25m 들렸다.

- 카메라 광학 프레임 주석이 0.25m 바닥을 광학 프레임 탓으로 설명하던 것 정정
- primitives 는 폐기 대상이라 값은 두고 같은 결함이 있음(+0.205m)만 명시
- tools/urdf_ground_check.py: URDF 만으로 바닥 높이를 검사 (ROS 불필요)
  수정 후 -0.002 OK / 수정 전 +0.248 FAIL / primitives +0.205 FAIL

File: src/drobot_description/urdf/drobot.urdf.xacro (robot description, xacro)
@@ -6,5 +6,5 @@
        - ROS1 catkin -> ROS2 ament, .urdf -> .urdf.xacro
        - mesh paths: package://drobot_description/meshes/
-       - base_footprint added (z=0.25 offset)
+       - base_footprint added (z=0 — 2026-10-02 에 0.25 에서 고침, 아래 BASE 참고)
        - left_rear_arm mass=0 -> 0.05 + min inertia
        - arm dynamics: damping=5.0 friction=1.0
@@ -22,9 +22,24 @@
   <material name="sensor_color"><color rgba="0.79 0.82 0.93 1"/></material>
   <!-- ==================== BASE ==================== -->
+  <!-- base_footprint 는 바퀴가 닿는 바닥면이어야 한다 (REP-120).
+       이 메시 모델은 base_link 원점이 이미 바닥 높이에 있다.
+       바퀴 접지점이 base_link 기준 z = -0.002(왼쪽) / +0.005(오른쪽) 이다
+       (tools/urdf_ground_check.py 로 STL 에서 계산).
+       그래서 오프셋은 0 이다.
+       예전 값 0.25 는 base_link 가 바닥에서 25 cm 위에 있다고 가정한 것이었다.
+       그러면 Gazebo 에서는 바퀴가 땅에 닿아야 하므로 base_footprint 가
+       땅 밑 -0.25 m 에 놓이는데 (실측 gz model z = -0.2518),
+       EKF(two_d_mode) 는 base_footprint 를 z=0 으로 고정한다.
+       그 결과 TF 를 거친 센서 점이 전부 0.25 m 들려서
+         - 빈 바닥이 0.25 m 로 측정됐고 (> rover_traversable_max 0.15 → fly_over)
+         - 카메라가 TF 상 0.61 m, 실제 0.36 m 라 0.5 m 장애물 윗면을 못 봤다.
+       남는 오차: 좌우 바퀴 메시가 7 mm 비대칭이라 로봇이 약 1.2° 기울어
+       놓인다 (실측 roll 0.021 rad). two_d_mode 는 이 기울기를 TF 에 넣지
+       않으므로 바닥이 옆으로 4 m 떨어진 곳에서 ±8 cm 정도 기울어 보인다. -->
   <link name="base_footprint"/>
   <joint name="base_footprint_joint" type="fixed">
     <parent link="base_footprint"/>
     <child link="base_link"/>
-    <origin xyz="0 0 0.25" rpy="0 0 0"/>
+    <origin xyz="0 0 0" rpy="0 0 0"/>
   </joint>
   <link name="base_link">
@@ -91,18 +106,12 @@
     <child link="camera_link"/>
   </joint>
-  <!-- 카메라 광학 프레임 (REP-103 / REP-145)
-       Gazebo 의 rgbd 센서는 포인트클라우드를 광학 좌표계로 낸다:
-           x 오른쪽 · y 아래 · z 전방
-       반면 camera_link 는 ROS 본체 좌표계다:
-           x 전방 · y 왼쪽 · z 위
-       둘을 같은 프레임으로 선언하면 축이 두 번 90도 어긋나, 바닥 점이
-       로봇 자신의 높이로 찍히고 장애물은 엉뚱한 자리에 쌓인다.
-       실제로 elevation_layer 가 빈 바닥 전 구간을 0.25 m(= base_link 높이)로
-       보고 0.5 m 장애물은 전혀 못 봤다. 2026-10-02 확인.
-       주의: gazebo.xacro 의 gz_frame_id 는 camera_link 를 쓴다.
-       Gazebo 가 내는 PointCloud2 는 이미 x 전방 규약이라
-       이 프레임을 가리키면 90도 회전이 두 번 들어가 점이 엉뚱한
-       방향으로 날아간다 (실측 확인). 이 링크는 다른 도구와의
-       호환을 위해 선언만 해 둔다. -->
+  <!-- 카메라 광학 프레임 (REP-103: x 오른쪽 · y 아래 · z 전방)
+       gazebo.xacro 의 gz_frame_id 는 이 프레임이 아니라 camera_link 를 쓴다.
+       Gazebo 가 내는 PointCloud2 는 이미 본체 규약(x 전방 · y 왼쪽 · z 위)이라
+       여기를 가리키면 회전이 한 번 더 들어가 점이 엉뚱한 방향으로 날아간다
+       (2026-10-02 실측: 점이 +y 대신 +x 로 갔다).
+       광학 규약을 기대하는 다른 도구와의 호환을 위해 선언만 해 둔다.
+       참고: 같은 날 '빈 바닥이 0.25 m 로 보인다' 를 이 프레임 탓으로 잘못
+       짚었었다. 원인은 base_footprint_joint 의 높이였다 (위 BASE 참고). -->
   <link name="camera_link_optical"/>
   <joint name="camera_optical_joint" type="fixed">

File: src/drobot_description/urdf/drobot_primitives.urdf.xacro (robot description, xacro)
@@ -9,4 +9,10 @@
        right_front_arm  collision/visual origin z = -0.175993  (좌우 비대칭)
      visual 뿐 아니라 collision 도 틀려서 물리가 어긋난다.
+     바닥 높이도 틀려 있다 (2026-10-02 확인, 고치지 않고 둔다):
+       base_footprint_joint z=0.25 인데 충돌체 최저점(base_link 박스)이
+       base_footprint 기준 +0.205 m 다. 그래서 TF 를 거친 센서 점이
+       0.2 m 쯤 들려 보이고, 빈 바닥이 fly_over 로 분류된다.
+       바퀴보다 몸체 박스가 4.8 cm 낮아 몸체가 바닥에 끌린다.
+       메시 모델은 drobot.urdf.xacro 에서 0 으로 고쳤다.
      급히 만든 대체본이었고, 고쳐 쓰기보다 원본 메시를 쓰는 편이 맞다.
      참고용으로만 남긴다.
@@ -114,18 +120,6 @@
     <child link="camera_link"/>
   </joint>
-  <!-- 카메라 광학 프레임 (REP-103 / REP-145)
-       Gazebo 의 rgbd 센서는 포인트클라우드를 광학 좌표계로 낸다:
-           x 오른쪽 · y 아래 · z 전방
-       반면 camera_link 는 ROS 본체 좌표계다:
-           x 전방 · y 왼쪽 · z 위
-       둘을 같은 프레임으로 선언하면 축이 두 번 90도 어긋나, 바닥 점이
-       로봇 자신의 높이로 찍히고 장애물은 엉뚱한 자리에 쌓인다.
-       실제로 elevation_layer 가 빈 바닥 전 구간을 0.25 m(= base_link 높이)로
-       보고 0.5 m 장애물은 전혀 못 봤다. 2026-10-02 확인.
-       주의: gazebo.xacro 의 gz_frame_id 는 camera_link 를 쓴다.
-       Gazebo 가 내는 PointCloud2 는 이미 x 전방 규약이라
-       이 프레임을 가리키면 90도 회전이 두 번 들어가 점이 엉뚱한
-       방향으로 날아간다 (실측 확인). 이 링크는 다른 도구와의
-       호환을 위해 선언만 해 둔다. -->
+  <!-- 카메라 광학 프레임 — 선언만 해 둔다.
+       gz_frame_id 는 camera_link 가 맞다. 이유는 drobot.urdf.xacro 의 같은 자리 주석 참고. -->
   <link name="camera_link_optical"/>
   <joint name="camera_optical_joint" type="fixed">
